File: esp32_hosted.kicad_sch (KiCad schematic)
At the start: 27 parts, among them J1 BT_UART, J2 WIFI, J3 PWR, J4 PROG, SW1 RESET, U1 AP7384-33SA, U2 ESP32-WROOM-32, U3 PCB_SD

Commit message: forgot to breakout the reset pin
Parts:
- removed J3: PWR, Connector_PinSocket_2.54mm:PinSocket_1x03_P2.54mm_Vertical, symbol Connector:Conn_01x03_Male
- added J3: PWR, Connector_PinSocket_2.54mm:PinSocket_1x04_P2.54mm_Vertical, symbol Connector:Conn_01x04_Male
Connections:
- net +3.3V: now also J3.3 (Pin_3)
- net +5V: now also J3.1 (Pin_1)
- net ESP_RTS: now also J3.4 (Pin_4)
- net GND: now also J3.2 (Pin_2)
Changed lines of the file:
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@@
+    (stroke (width 0) (type default) (color 0 0 0 0))
+  )
+  (wire (pts (xy 51.054 59.436) (xy 53.086 59.436))
     (stroke (width 0) (type default) (color 0 0 0 0))
   )
@@
     (stroke (width 0) (type default) (color 0 0 0 0))
   )
+  (wire (pts (xy 53.086 67.818) (xy 53.086 59.436))
+    (stroke (width 0) (type default) (color 0 0 0 0))
+  )
   (wire (pts (xy 82.804 24.384) (xy 82.804 26.416))
     (stroke (width 0) (type default) (color 0 0 0 0))
@@
     (stroke (width 0) (type default) (color 0 0 0 0))
   )
-  (wire (pts (xy 54.102 65.278) (xy 54.102 56.896))
+  (wire (pts (xy 54.102 56.896) (xy 54.102 69.088))
     (stroke (width 0) (type default) (color 0 0 0 0))
   )
@@
     (stroke (width 0) (type default) (color 0 0 0 0))
   )
-  (wire (pts (xy 48.768 64.516) (xy 48.768 65.278))
+  (wire (pts (xy 48.006 68.326) (xy 48.006 69.088))
     (stroke (width 0) (type default) (color 0 0 0 0))
   )
@@
     (stroke (width 0) (type default) (color 0 0 0 0))
   )
-  (wire (pts (xy 48.768 65.278) (xy 54.102 65.278))
+  (wire (pts (xy 48.006 69.088) (xy 54.102 69.088))
     (stroke (width 0) (type default) (color 0 0 0 0))
   )
@@
   )
   (label "D2{slash}MISO" (at 85.09 141.224 0)
+    (effects (font (size 1.27 1.27)) (justify left bottom))
+  )
+  (label "ESP_RTS" (at 53.086 67.818 90)
     (effects (font (size 1.27 1.27)) (justify left bottom))
   )
@@
     (pin "5")
     (pin "6")
-  )
-  (symbol (lib_id "Connector:Conn_01x03_Male") (at 45.974 54.356 0) (unit 1)
-    (in_bom yes) (on_board yes)
-    (property "Reference" "J3" (id 0) (at 43.688 51.816 0))
-    (property "Value" "PWR" (id 1) (at 43.688 54.356 0))
-    (property "Footprint" "Connector_PinSocket_2.54mm:PinSocket_1x03_P2.54mm_Vertical" (id 2) (at 45.974 54.356 0)
-      (effects (font (size 1.27 1.27)) hide)
-    )
-    (property "Datasheet" "~" (id 3) (at 45.974 54.356 0)
-      (effects (font (size 1.27 1.27)) hide)
-    )
-    (pin "1")
-    (pin "2")
-    (pin "3")
   )
   (symbol (lib_id "Device:R") (at 97.282 84.836 0) (unit 1)
@@
     (pin "2")
   )
-  (symbol (lib_id "power:+3.3V") (at 48.768 64.516 0) (unit 1)
-    (in_bom yes) (on_board yes) (fields_autoplaced)
-    (property "Reference" "#PWR0102" (id 0) (at 48.768 68.326 0)
-      (effects (font (size 1.27 1.27)) hide)
-    )
-    (property "Value" "+3.3V" (id 1) (at 48.768 59.182 0))
-    (property "Footprint" "" (id 2) (at 48.768 64.516 0)
-      (effects (font (size 1.27 1.27)) hide)
-    )
-    (property "Datasheet" "" (id 3) (at 48.768 64.516 0)
+  (symbol (lib_id "power:+3.3V") (at 48.006 68.326 0) (unit 1)
+    (in_bom yes) (on_board yes)
+    (property "Reference" "#PWR0102" (id 0) (at 48.006 72.136 0)
+      (effects (font (size 1.27 1.27)) hide)
+    )
+    (property "Value" "+3.3V" (id 1) (at 48.006 62.992 0))
+    (property "Footprint" "" (id 2) (at 48.006 68.326 0)
+      (effects (font (size 1.27 1.27)) hide)
+    )
+    (property "Datasheet" "" (id 3) (at 48.006 68.326 0)
       (effects (font (size 1.27 1.27)) hide)
     )
@@
     )
     (pin "1")
+  )
+  (symbol (lib_id "Connector:Conn_01x04_Male") (at 45.974 54.356 0) (unit 1)
+    (in_bom yes) (on_board yes)
+    (property "Reference" "J3" (id 0) (at 43.434 51.816 0))
+    (property "Value" "PWR" (id 1) (at 43.434 54.356 0))
+    (property "Footprint" "Connector_PinSocket_2.54mm:PinSocket_1x04_P2.54mm_Vertical" (id 2) (at 45.974 54.356 0)
+      (effects (font (size 1.27 1.27)) hide)
+    )
+    (property "Datasheet" "~" (id 3) (at 45.974 54.356 0)
+      (effects (font (size 1.27 1.27)) hide)
+    )
+    (pin "1")
+    (pin "2")
+    (pin "3")
+    (pin "4")
   )
   (symbol (lib_id "power:+3.3V") (at 97.282 78.994 0) (unit 1)
@@
       (reference "J2") (unit 1) (value "WIFI") (footprint "Connector_PinSocket_2.54mm:PinSocket_1x08_P2.54mm_Vertical")
     )
-    (path "/1aa6fa02-2466-431a-9afd-f1934871be5a"
-      (reference "J3") (unit 1) (value "PWR") (footprint "Connector_PinSocket_2.54mm:PinSocket_1x03_P2.54mm_Vertical")
+    (path "/e6c886c3-fe40-45c8-8cb4-ed709ece738c"
+      (reference "J3") (unit 1) (value "PWR") (footprint "Connector_PinSocket_2.54mm:PinSocket_1x04_P2.54mm_Vertical")
     )
     (path "/174f2c1e-484c-4ed7-b695-3cf0a93b1112"
